File: comparator/comparator.kicad_pcb (KiCad board)
At the start: 4 copper layers, 55.9 x 22.9 mm, 54 parts, among them J1 PMOD, J10 SMA, J11 DC Block, J12 50R Term/Ref, J20 SMA, J21 DC Block, J22 50R Term/Ref, U30 LT1711xMS8, U40 LM2776, U51 LM4040DBZ-2.5, U52 LM4040DBZ-2.5

Commit message: Finished ground stitching vias
Routing:
- net /VCC_N: track 65.8 -> 63.3 mm
- net GND: vias 86 -> 119
Other:
- board text added: "Layers: 4 PCB Thickness: 1.6mm Mask Colour: Green Surface Finish: ENIG-RoHS Copper Weight: 1oz Material: FR4 Tented vias"
- board text removed: "Layers: 2 PCB Thickness: 1.6mm Mask Colour: Green Surface Finish: ENIG-RoHS Copper Weight: 1oz Material: FR4 Tented vias"
Changed lines of the file:
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@@
     (thickness 1.6)
     (drawings 20)
-    (tracks 281)
+    (tracks 315)
     (zones 0)
     (modules 54)
@@
     (effects (font (size 0.762 0.762) (thickness 0.0762)))
   )
-  (gr_text "Layers: 2\nPCB Thickness: 1.6mm\nMask Colour: Green\nSurface Finish: ENIG-RoHS\nCopper Weight: 1oz\nMaterial: FR4\n\nTented vias" (at 174.879 128.143) (layer Cmts.User)
+  (gr_text "Layers: 4\nPCB Thickness: 1.6mm\nMask Colour: Green\nSurface Finish: ENIG-RoHS\nCopper Weight: 1oz\nMaterial: FR4\n\nTented vias" (at 191.389 98.044) (layer Cmts.User)
     (effects (font (size 1.5 1.5) (thickness 0.3)) (justify left))
   )
@@
   (via (at 125.857 95.25) (size 0.8) (drill 0.4) (layers F.Cu B.Cu) (net 1))
   (via (at 125.857 89.916) (size 0.8) (drill 0.4) (layers F.Cu B.Cu) (net 1))
+  (via (at 128.27 108.585) (size 0.8) (drill 0.4) (layers F.Cu B.Cu) (net 1))
+  (via (at 131.445 108.585) (size 0.8) (drill 0.4) (layers F.Cu B.Cu) (net 1))
+  (via (at 134.62 108.585) (size 0.8) (drill 0.4) (layers F.Cu B.Cu) (net 1))
+  (via (at 137.795 108.585) (size 0.8) (drill 0.4) (layers F.Cu B.Cu) (net 1))
+  (via (at 140.97 108.585) (size 0.8) (drill 0.4) (layers F.Cu B.Cu) (net 1))
+  (via (at 144.145 108.585) (size 0.8) (drill 0.4) (layers F.Cu B.Cu) (net 1))
+  (via (at 147.32 108.585) (size 0.8) (drill 0.4) (layers F.Cu B.Cu) (net 1))
+  (via (at 150.495 108.585) (size 0.8) (drill 0.4) (layers F.Cu B.Cu) (net 1))
+  (via (at 159.385 108.585) (size 0.8) (drill 0.4) (layers F.Cu B.Cu) (net 1))
+  (via (at 162.56 108.585) (size 0.8) (drill 0.4) (layers F.Cu B.Cu) (net 1))
+  (via (at 165.735 108.585) (size 0.8) (drill 0.4) (layers F.Cu B.Cu) (net 1))
+  (via (at 168.91 108.585) (size 0.8) (drill 0.4) (layers F.Cu B.Cu) (net 1))
+  (via (at 159.385 86.995) (size 0.8) (drill 0.4) (layers F.Cu B.Cu) (net 1))
+  (via (at 162.56 86.995) (size 0.8) (drill 0.4) (layers F.Cu B.Cu) (net 1))
+  (via (at 165.735 86.995) (size 0.8) (drill 0.4) (layers F.Cu B.Cu) (net 1))
+  (via (at 168.91 86.995) (size 0.8) (drill 0.4) (layers F.Cu B.Cu) (net 1))
+  (via (at 164.465 91.44) (size 0.8) (drill 0.4) (layers F.Cu B.Cu) (net 1))
+  (via (at 164.465 93.98) (size 0.8) (drill 0.4) (layers F.Cu B.Cu) (net 1))
+  (via (at 171.45 93.98) (size 0.8) (drill 0.4) (layers F.Cu B.Cu) (net 1))
+  (via (at 171.45 91.44) (size 0.8) (drill 0.4) (layers F.Cu B.Cu) (net 1))
+  (via (at 164.465 101.6) (size 0.8) (drill 0.4) (layers F.Cu B.Cu) (net 1))
+  (via (at 164.465 104.14) (size 0.8) (drill 0.4) (layers F.Cu B.Cu) (net 1))
+  (via (at 171.45 101.6) (size 0.8) (drill 0.4) (layers F.Cu B.Cu) (net 1))
+  (via (at 171.45 104.14) (size 0.8) (drill 0.4) (layers F.Cu B.Cu) (net 1))
+  (via (at 158.877 97.79) (size 0.8) (drill 0.4) (layers F.Cu B.Cu) (net 1))
+  (via (at 158.115 94.234) (size 0.8) (drill 0.4) (layers F.Cu B.Cu) (net 1))
+  (via (at 158.115 101.6) (size 0.8) (drill 0.4) (layers F.Cu B.Cu) (net 1))
+  (via (at 147.193 99.441) (size 0.8) (drill 0.4) (layers F.Cu B.Cu) (net 1))
+  (via (at 147.193 96.393) (size 0.8) (drill 0.4) (layers F.Cu B.Cu) (net 1))
+  (via (at 131.318 92.71) (size 0.8) (drill 0.4) (layers F.Cu B.Cu) (net 1))
+  (via (at 129.032 95.758) (size 0.8) (drill 0.4) (layers F.Cu B.Cu) (net 1))
+  (via (at 130.175 94.234) (size 0.8) (drill 0.4) (layers F.Cu B.Cu) (net 1))
+  (via (at 148.971 97.282) (size 0.8) (drill 0.4) (layers F.Cu B.Cu) (net 1))
   (segment (start 124.46 103.505) (end 123.825 104.14) (width 0.5) (layer F.Cu) (net 2))
   (segment (start 127.505 103.505) (end 124.46 103.505) (width 0.5) (layer F.Cu) (net 2))
@@
   (segment (start 151.257 101.473) (end 151.257 107.823) (width 0.25) (layer In2.Cu) (net 10))
   (segment (start 151.257 107.823) (end 152.019 108.585) (width 0.25) (layer In2.Cu) (net 10))
-  (segment (start 158.242 108.007002) (end 158.242 96.52) (width 0.25) (layer In2.Cu) (net 10))
-  (segment (start 158.078001 96.356001) (end 155.575 93.853) (width 0.25) (layer In2.Cu) (net 10))
-  (segment (start 158.242 96.52) (end 158.078001 96.356001) (width 0.25) (layer In2.Cu) (net 10))
-  (segment (start 153.416 108.585) (end 157.664002 108.585) (width 0.25) (layer In2.Cu) (net 10))
-  (segment (start 157.664002 108.585) (end 158.242 108.007002) (width 0.25) (layer In2.Cu) (net 10))
   (segment (start 140.97 101.473) (end 151.257 101.473) (width 0.25) (layer In2.Cu) (net 10))
   (segment (start 137.414 94.361) (end 137.414 97.917) (width 0.25) (layer In2.Cu) (net 10))
@@
   (segment (start 152.019 108.585) (end 153.289 108.585) (width 0.25) (layer In2.Cu) (net 10))
   (segment (start 153.289 108.585) (end 153.416 108.585) (width 0.25) (layer In2.Cu) (net 10))
+  (segment (start 155.251002 108.585) (end 155.067 108.585) (width 0.25) (layer In2.Cu) (net 10))
+  (segment (start 156.877999 95.721684) (end 156.877999 106.958003) (width 0.25) (layer In2.Cu) (net 10))
+  (segment (start 155.575 93.853) (end 155.575 94.418685) (width 0.25) (layer In2.Cu) (net 10))
+  (segment (start 156.877999 106.958003) (end 155.251002 108.585) (width 0.25) (layer In2.Cu) (net 10))
+  (segment (start 155.575 94.418685) (end 156.877999 95.721684) (width 0.25) (layer In2.Cu) (net 10))
+  (segment (start 153.416 108.585) (end 155.067 108.585) (width 0.25) (layer In2.Cu) (net 10))
   (segment (start 138.4555 102.946) (end 138.43 102.9715) (width 0.25) (layer F.Cu) (net 11))
   (segment (start 138.4555 101.473) (end 138.4555 102.946) (width 0.25) (layer F.Cu) (net 11))

Commit message: Released Rev 09/09/19 first manufacture
Parts:
- R31, R32: value 270 -> 330
Other:
- board text added: "09/09/2019"
- board text removed: "21/06/2019"
Changed lines of the file:
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@@
       (linewidth 0.100000)
       (plotframeref false)
-      (viasonmask true)
+      (viasonmask false)
       (mode 1)
       (useauxorigin false)
@@
       (effects (font (size 0.762 0.762) (thickness 0.0762)))
     )
-    (fp_text value 270 (at 0 1.016) (layer F.Fab)
+    (fp_text value 330 (at 0 1.016) (layer F.Fab)
       (effects (font (size 0.508 0.508) (thickness 0.0508)))
     )
@@
       (effects (font (size 0.762 0.762) (thickness 0.0762)))
     )
-    (fp_text value 270 (at 0 1.016) (layer F.Fab)
+    (fp_text value 330 (at 0 1.016) (layer F.Fab)
       (effects (font (size 0.508 0.508) (thickness 0.0508)))
     )
@@
   )
   (gr_poly (pts (xy 125.095 86.36) (xy 125.095 87.63) (xy 153.035 87.63) (xy 153.035 86.36)) (layer B.Mask) (width 0.1))
-  (gr_text 21/06/2019 (at 132.334 96.139) (layer F.SilkS)
+  (gr_text 09/09/2019 (at 132.334 96.139) (layer F.SilkS)
     (effects (font (size 0.762 0.762) (thickness 0.0762)))
   )
