File: comparator/comparator.sch (KiCad schematic (older format))
At the start: 54 parts, among them J1 PMOD, J10 SMA, J11 DC Block, J12 50R Term/Ref, J20 SMA, J21 DC Block, J22 50R Term/Ref, U30 LT1711xMS8, U40 LM2776, U51 LM4040DBZ-2.5, U52 LM4040DBZ-2.5

Commit message: Released Rev 09/09/19 first manufacture
Parts:
- R31, R32: value 270 -> 330
Changed lines of the file:
@@
 Sheet 1 1
 Title "emods/comparator"
-Date "2019-08-13"
-Rev "13/08/19"
+Date "2019-09-09"
+Rev "09/09/19"
 Comp "cpgmoore"
-Comment1 "REV 13/08/19 - Work in progress"
+Comment1 "REV 09/09/19 - First Manufacture"
 Comment2 ""
 Comment3 ""
@@
 P 1350 950
 F 0 "R31" V 1250 950 50  0000 R CNN
-F 1 "270" V 1250 1150 50  0000 R CNN
+F 1 "330" V 1250 1150 50  0000 R CNN
 F 2 "Resistor_SMD:R_0603_1608Metric" H 1350 950 50  0001 C CNN
 F 3 "~" H 1350 950 50  0001 C CNN
@@
 P 1350 1050
 F 0 "R32" V 1450 1050 50  0000 R CNN
-F 1 "270" V 1450 1250 50  0000 R CNN
+F 1 "330" V 1450 1250 50  0000 R CNN
 F 2 "Resistor_SMD:R_0603_1608Metric" H 1350 1050 50  0001 C CNN
 F 3 "~" H 1350 1050 50  0001 C CNN
@@
 $EndComp
 $Comp
-L power:GND #PWR?
+L power:GND #PWR0101
 U 1 1 5D661185
 P 3550 2750
-F 0 "#PWR?" H 3550 2500 50  0001 C CNN
+F 0 "#PWR0101" H 3550 2500 50  0001 C CNN
 F 1 "GND" H 3555 2577 50  0000 C CNN
 F 2 "" H 3550 2750 50  0001 C CNN
